File: circuits/chandelier/fixed.kicad_sch (KiCad schematic)
At the start: 8 parts

Commit message: Structure: circuits/, lib/, tools/, build/<circuit>/
Circuit models moved to circuits/<circuit>/<variant>.kicad_sch, model
library to lib/spice/models.lib, scripts to tools/ with shared code in
tools/circuit_tools/. Output files go to build/<circuit>/. A variant is
a .kicad_sch with a .kicad_pro of the same name, so KiCad autosaves are
skipped. Python project renamed to circuit_lab. Documentation updated.

Also marks stage 1 of task 0002 as done.
Connections:
- net GND: now also LA1.1 (-), LA2.1 (-), LA3.1 (-), LA4.1 (-), LA5.1 (-); no longer LA1.2 (+), LA2.2 (+)
- removed net X_BLUE: B1.2 (B), LA1.1 (-), LA2.1 (-), LA3.1 (-), LA4.1 (-), LA5.1 (-)
- new net X_BR2: B1.2 (B), LA1.2 (+), LA2.2 (+)
Other:
- note added: "Люстра — как должно быть"
- note removed: "Люстра — как есть (гипотеза)"
- note removed: "ОШИБКА: фаза B1 и N"
- note removed: "перепутаны на X_BLUE и X_BR2"
